Commit message: added imu, removed src and executable from CMAKE

File: src/qcar_gazebo/urdf/qcar_model.xacro (robot description, xacro)
@@ -1,8 +1,9 @@
 <?xml version='1.0'?>
 <robot name="QCar" xmlns:xacro="http://www.ros.org/wiki/xacro">
-  <xacro:include filename="$(find mybot_gazebo)/urdf/materials.xacro" />
-  <!-- <xacro:include filename="$(find mybot_gazebo)/urdf/lidar.xacro" /> -->
-  <!-- <xacro:include filename="$(find mybot_gazebo)/urdf/camera.xacro" /> -->
-  <!-- <xacro:include filename="$(find mybot_gazebo)/urdf/depth_camera.xacro" /> -->
+  <xacro:include filename="$(find qcar_gazebo)/urdf/materials.xacro" />
+  <!-- <xacro:include filename="$(find qcar_gazebo)/urdf/lidar.xacro" /> -->
+  <!-- <xacro:include filename="$(find qcar_gazebo)/urdf/camera.xacro" /> -->
+  <!-- <xacro:include filename="$(find qcar_gazebo)/urdf/depth_camera.xacro" /> -->
+  <!-- <xacro:include filename="$(find qcar_gazebo)/urdf/imu.xacro" /> -->
   <link name="base_footprint"/>
   <joint name="base_joint" type="fixed">
@@ -14,5 +15,5 @@
             <origin rpy="0 0 0" xyz="0 0 0"/>
             <geometry>
-                <mesh filename="package://mybot_gazebo/models/qcar/QCarBody.stl" scale="0.001 0.001 0.001"/>
+                <mesh filename="package://qcar_gazebo/models/qcar/QCarBody.stl" scale="0.001 0.001 0.001"/>
             </geometry>
             <material name="white"/>
@@ -21,5 +22,5 @@
             <origin rpy="0 0 0" xyz="0 0 0"/>
             <geometry>
-                <mesh filename="package://mybot_gazebo/models/qcar/QCarBody.stl" scale="0.001 0.001 0.001"/>
+                <mesh filename="package://qcar_gazebo/models/qcar/QCarBody.stl" scale="0.001 0.001 0.001"/>
             </geometry>
         </collision>
@@ -40,5 +41,5 @@
             <origin rpy="0 0 0" xyz="0 0 0"/>
             <geometry>
-                <mesh filename="package://mybot_gazebo/models/qcar/QCarLidar.stl" scale="0.001 0.001 0.001"/>
+                <mesh filename="package://qcar_gazebo/models/qcar/QCarLidar.stl" scale="0.001 0.001 0.001"/>
             </geometry>
             <material name="red"/>
@@ -47,5 +48,5 @@
             <origin rpy="0 0 0" xyz="0 0 0"/>
             <geometry>
-                <mesh filename="package://mybot_gazebo/models/qcar/QCarLidar.stl" scale="0.001 0.001 0.001"/>
+                <mesh filename="package://qcar_gazebo/models/qcar/QCarLidar.stl" scale="0.001 0.001 0.001"/>
             </geometry>
         </collision>
@@ -69,5 +70,5 @@
             <origin rpy="0 0 0" xyz="0 0 0"/>
             <geometry>
-                <mesh filename="package://mybot_gazebo/models/qcar/QCarSteeringHubL.stl" scale="0.001 0.001 0.001"/>
+                <mesh filename="package://qcar_gazebo/models/qcar/QCarSteeringHubL.stl" scale="0.001 0.001 0.001"/>
             </geometry>
             <material name="orange"/>
@@ -76,5 +77,5 @@
             <origin rpy="0 0 0" xyz="0 0 0"/>
             <geometry>
-                <mesh filename="package://mybot_gazebo/models/qcar/QCarSteeringHubL.stl" scale="0.001 0.001 0.001"/>
+                <mesh filename="package://qcar_gazebo/models/qcar/QCarSteeringHubL.stl" scale="0.001 0.001 0.001"/>
             </geometry>
         </collision>
@@ -98,5 +99,5 @@
             <origin rpy="0 0 0" xyz="0 0 0"/>
             <geometry>
-                <mesh filename="package://mybot_gazebo/models/qcar/QCarSteeringHubR.stl" scale="0.001 0.001 0.001"/>
+                <mesh filename="package://qcar_gazebo/models/qcar/QCarSteeringHubR.stl" scale="0.001 0.001 0.001"/>
             </geometry>
             <material name="orange"/>
@@ -105,5 +106,5 @@
             <origin rpy="0 0 0" xyz="0 0 0"/>
             <geometry>
-                <mesh filename="package://mybot_gazebo/models/qcar/QCarSteeringHubR.stl" scale="0.001 0.001 0.001"/>
+                <mesh filename="package://qcar_gazebo/models/qcar/QCarSteeringHubR.stl" scale="0.001 0.001 0.001"/>
             </geometry>
         </collision>
@@ -124,5 +125,5 @@
             <origin rpy="0 0 0" xyz="0 0 0"/>
             <geometry>
-                <mesh filename="package://mybot_gazebo/models/qcar/QCarWheel.stl" scale="0.001 0.001 0.001"/>
+                <mesh filename="package://qcar_gazebo/models/qcar/QCarWheel.stl" scale="0.001 0.001 0.001"/>
             </geometry>
             <material name="red"/>
@@ -131,5 +132,5 @@
             <origin rpy="0 0 0" xyz="0 0 0"/>
             <geometry>
-                <mesh filename="package://mybot_gazebo/models/qcar/QCarWheel.stl" scale="0.001 0.001 0.001"/>
+                <mesh filename="package://qcar_gazebo/models/qcar/QCarWheel.stl" scale="0.001 0.001 0.001"/>
             </geometry>
         </collision>
@@ -150,5 +151,5 @@
             <origin rpy="0 0 0" xyz="0 0 0"/>
             <geometry>
-                <mesh filename="package://mybot_gazebo/models/qcar/QCarWheel.stl" scale="0.001 0.001 0.001"/>
+                <mesh filename="package://qcar_gazebo/models/qcar/QCarWheel.stl" scale="0.001 0.001 0.001"/>
             </geometry>
             <material name="orange"/>
@@ -157,5 +158,5 @@
             <origin rpy="0 0 0" xyz="0 0 0"/>
             <geometry>
-                <mesh filename="package://mybot_gazebo/models/qcar/QCarWheel.stl" scale="0.001 0.001 0.001"/>
+                <mesh filename="package://qcar_gazebo/models/qcar/QCarWheel.stl" scale="0.001 0.001 0.001"/>
             </geometry>
         </collision>
@@ -176,5 +177,5 @@
             <origin rpy="0 0 0" xyz="0 0 0"/>
             <geometry>
-                <mesh filename="package://mybot_gazebo/models/qcar/QCarWheel.stl" scale="0.001 0.001 0.001"/>
+                <mesh filename="package://qcar_gazebo/models/qcar/QCarWheel.stl" scale="0.001 0.001 0.001"/>
             </geometry>
             <material name="orange"/>
@@ -183,5 +184,5 @@
             <origin rpy="0 0 0" xyz="0 0 0"/>
             <geometry>
-                <mesh filename="package://mybot_gazebo/models/qcar/QCarWheel.stl" scale="0.001 0.001 0.001"/>
+                <mesh filename="package://qcar_gazebo/models/qcar/QCarWheel.stl" scale="0.001 0.001 0.001"/>
             </geometry>
         </collision>
@@ -202,5 +203,5 @@
             <origin rpy="0 0 0" xyz="0 0 0"/>
             <geometry>
-                <mesh filename="package://mybot_gazebo/models/qcar/QCarWheel.stl" scale="0.001 0.001 0.001"/>
+                <mesh filename="package://qcar_gazebo/models/qcar/QCarWheel.stl" scale="0.001 0.001 0.001"/>
             </geometry>
             <material name="red"/>
@@ -209,5 +210,5 @@
             <origin rpy="0 0 0" xyz="0 0 0"/>
             <geometry>
-                <mesh filename="package://mybot_gazebo/models/qcar/QCarWheel.stl" scale="0.001 0.001 0.001"/>
+                <mesh filename="package://qcar_gazebo/models/qcar/QCarWheel.stl" scale="0.001 0.001 0.001"/>
             </geometry>
         </collision>

Commit message: Integrated motor joints. Track1.launch adjusted.

File: src/qcar_gazebo/urdf/qcar_model.xacro (robot description, xacro)
@@ -116,10 +116,15 @@
         </inertial>
     </link>
-    <joint name="hubfl_wheelfl_joint" type="continuous">
+    <!-- <joint name="hubfl_wheelfl_joint" type="continuous">
         <parent link="hubfl"/>
         <child link="wheelfl"/>
         <origin rpy="0 0 3.14" xyz="0 0 0"/>
         <axis xyz="0 1 0"/>
-    </joint>
+    </joint> -->
+    <xacro:joint_motor motor_name="wheelfl_motor" parent_link="hubfl" child_link="wheelfl">
+        <xacro:property name="params_yaml" value="$(find gazebo_ros_motors)/params/joint_motor.yaml"/>
+        <origin xyz="0 0 0" rpy="0 0 3.14"/>
+        <axis xyz="0 1 0" rpy="0 0 0"/>
+    </xacro:joint_motor>
     <link name="wheelfl">
         <visual>
@@ -142,10 +147,15 @@
         </inertial>
     </link>
-    <joint name="hubfr_wheelfr_joint" type="continuous">
+    <!-- <joint name="hubfr_wheelfr_joint" type="continuous">
         <parent link="hubfr"/>
         <child link="wheelfr"/>
         <origin rpy="0 0 0" xyz="0 0 0"/>
         <axis xyz="0 1 0"/>
-    </joint>
+    </joint> -->
+    <xacro:joint_motor motor_name="wheelfr_motor" parent_link="hubfr" child_link="wheelfr">
+        <xacro:property name="params_yaml" value="$(find gazebo_ros_motors)/params/joint_motor.yaml"/>
+        <origin xyz="0 0 0" rpy="0 0 0"/>
+        <axis xyz="0 1 0" rpy="0 0 0"/>
+    </xacro:joint_motor>
     <link name="wheelfr">
         <visual>
@@ -168,10 +178,15 @@
         </inertial>
     </link>
-    <joint name="base_wheelrl_joint" type="continuous">
+    <!-- <joint name="base_wheelrl_joint" type="continuous">
         <parent link="base"/>
         <child link="wheelrl"/>
         <origin rpy="0 0 3.14" xyz="-0.12765 0.05610 0.03338"/>
         <axis xyz="0 1 0"/>
-    </joint>
+    </joint> -->
+    <xacro:joint_motor motor_name="wheelrl_motor" parent_link="base" child_link="wheelrl">
+        <xacro:property name="params_yaml" value="$(find gazebo_ros_motors)/params/joint_motor.yaml"/>
+        <origin xyz="-0.12765 0.05610 0.03338" rpy="0 0 3.14"/>
+        <axis xyz="0 1 0" rpy="0 0 0"/>
+    </xacro:joint_motor>
     <link name="wheelrl">
         <visual>
@@ -194,10 +209,15 @@
         </inertial>
     </link>
-    <joint name="base_wheelrr_joint" type="continuous">
+    <!-- <joint name="base_wheelrr_joint" type="continuous">
         <parent link="base"/>
         <child link="wheelrr"/>
         <origin rpy="0 0 0" xyz="-0.12765 -0.05610 0.03338"/>
         <axis xyz="0 1 0"/>
-    </joint>
+    </joint> -->
+    <xacro:joint_motor motor_name="wheelrr_motor" parent_link="base" child_link="wheelrr">
+        <xacro:property name="params_yaml" value="$(find gazebo_ros_motors)/params/joint_motor.yaml"/>
+        <origin xyz="-0.12765 -0.05610 0.03338" rpy="0 0 0"/>
+        <axis xyz="0 1 0" rpy="0 0 0"/>
+    </xacro:joint_motor>
     <link name="wheelrr">
         <visual>
@@ -317,5 +337,5 @@
     <transmission name="hubfl_wheelfl_tran">
         <type>>transmission_interface/SimpleTransmission</type>
-        <joint name="hubfl_wheelfl_joint">
+        <joint name="wheelfl_motor">
             <hardwareInterface>hardware_interface/EffortJointInterface</hardwareInterface>
         </joint>
@@ -326,26 +346,8 @@
     <transmission name="hubfr_wheelfr_tran">
         <type>>transmission_interface/SimpleTransmission</type>
-        <joint name="hubfr_wheelfr_joint">
+        <joint name="wheelfr_motor">
             <hardwareInterface>hardware_interface/EffortJointInterface</hardwareInterface>
         </joint>
         <actuator name="hubfr_wheelfr_motor">
-            <mechanicalReduction>1</mechanicalReduction>
-        </actuator>
-    </transmission>
-    <transmission name="base_wheelrl_tran">
-        <type>>transmission_interface/SimpleTransmission</type>
-        <joint name="base_wheelrl_joint">
-            <hardwareInterface>hardware_interface/VelocityJointInterface</hardwareInterface>
-        </joint>
-        <actuator name="base_wheelrl_motor">
-            <mechanicalReduction>1</mechanicalReduction>
-        </actuator>
-    </transmission>
-    <transmission name="base_wheelrr_tran">
-        <type>>transmission_interface/SimpleTransmission</type>
-        <joint name="base_wheelrr_joint">
-            <hardwareInterface>hardware_interface/VelocityJointInterface</hardwareInterface>
-        </joint>
-        <actuator name="base_wheelrr_motor">
             <mechanicalReduction>1</mechanicalReduction>
         </actuator>

Commit message: added roscpp examples w/ comments

File: src/qcar_gazebo/urdf/qcar_model.xacro (robot description, xacro)
@@ -3,4 +3,5 @@
   <xacro:include filename="$(find qcar_gazebo)/urdf/materials.xacro" />
   <xacro:include filename="$(find gazebo_ros_motors)/xacro/joint_motor.xacro"/>
+  <xacro:include filename="$(find gazebo_ros_motors)/xacro/dc_motor.xacro"/> <!--dc motor plugin include-->
   <!-- <xacro:include filename="$(find qcar_gazebo)/urdf/lidar.xacro" /> -->
   <!-- <xacro:include filename="$(find qcar_gazebo)/urdf/camera.xacro" /> -->
@@ -116,10 +117,4 @@
         </inertial>
     </link>
-    <!-- <joint name="hubfl_wheelfl_joint" type="continuous">
-        <parent link="hubfl"/>
-        <child link="wheelfl"/>
-        <origin rpy="0 0 3.14" xyz="0 0 0"/>
-        <axis xyz="0 1 0"/>
-    </joint> -->
     <xacro:joint_motor motor_name="wheelfl_motor" parent_link="hubfl" child_link="wheelfl">
         <xacro:property name="params_yaml" value="$(find gazebo_ros_motors)/params/joint_motor.yaml"/>
@@ -147,10 +142,4 @@
         </inertial>
     </link>
-    <!-- <joint name="hubfr_wheelfr_joint" type="continuous">
-        <parent link="hubfr"/>
-        <child link="wheelfr"/>
-        <origin rpy="0 0 0" xyz="0 0 0"/>
-        <axis xyz="0 1 0"/>
-    </joint> -->
     <xacro:joint_motor motor_name="wheelfr_motor" parent_link="hubfr" child_link="wheelfr">
         <xacro:property name="params_yaml" value="$(find gazebo_ros_motors)/params/joint_motor.yaml"/>
@@ -178,10 +167,4 @@
         </inertial>
     </link>
-    <!-- <joint name="base_wheelrl_joint" type="continuous">
-        <parent link="base"/>
-        <child link="wheelrl"/>
-        <origin rpy="0 0 3.14" xyz="-0.12765 0.05610 0.03338"/>
-        <axis xyz="0 1 0"/>
-    </joint> -->
     <xacro:joint_motor motor_name="wheelrl_motor" parent_link="base" child_link="wheelrl">
         <xacro:property name="params_yaml" value="$(find gazebo_ros_motors)/params/joint_motor.yaml"/>
@@ -209,10 +192,4 @@
         </inertial>
     </link>
-    <!-- <joint name="base_wheelrr_joint" type="continuous">
-        <parent link="base"/>
-        <child link="wheelrr"/>
-        <origin rpy="0 0 0" xyz="-0.12765 -0.05610 0.03338"/>
-        <axis xyz="0 1 0"/>
-    </joint> -->
     <xacro:joint_motor motor_name="wheelrr_motor" parent_link="base" child_link="wheelrr">
         <xacro:property name="params_yaml" value="$(find gazebo_ros_motors)/params/joint_motor.yaml"/>

Commit message: Removed test limits

File: src/qcar_gazebo/urdf/qcar_model.xacro (robot description, xacro)
@@ -66,5 +66,4 @@
         <dynamics damping="0.143" friction="0.0"/>
         <limit lower="-0.5236" upper="0.5236" effort="300" velocity="2"/>
-        <!-- <limit lower="-3.1416" upper="3.1416" effort="300" velocity="2"/> -->
     </joint>
     <link name="hubfl">
@@ -94,5 +93,4 @@
         <axis xyz="0 0 1"/>
         <limit lower="-0.5236" upper="0.5236" effort="300" velocity="2"/>
-        <!-- <limit lower="-3.1416" upper="3.1416" effort="300" velocity="2"/> -->
         <dynamics damping="0.143" friction="0.0"/>
     </joint>
